Commit message: drive robot

File: description/robot.urdf.xacro (robot description, xacro)
@@ -2,3 +2,4 @@
 <robot xmlns:xacro="http://www.ros.org/wiki/xacro"  name="robot">
     <xacro:include filename = "robot_core.xacro"/>
+    <xacro:include filename = "gazebo_control.xacro"/>
 </robot>

File: description/robot_core.xacro (robot description, xacro)
@@ -39,4 +39,7 @@
     </xacro:inertial_box>
 </link>
+<gazebo reference="chassis">
+    <material>Gazebo/White</material>
+</gazebo>
 <!-- LEFT WHEEL -->
 <joint name="left_wheel_joint" type="continuous">
@@ -62,4 +65,7 @@
     </xacro:inertial_cylinder>
 </link>
+<gazebo reference="left_wheel">
+    <material>Gazebo/Blue</material>
+</gazebo>
 <!-- RIGHT WHEEL -->
 <joint name="right_wheel_joint" type="continuous">
@@ -85,4 +91,7 @@
     </xacro:inertial_cylinder>
 </link>
+<gazebo reference="right_wheel">
+    <material>Gazebo/Blue</material>
+</gazebo>
 <!-- CASTER WHEEL -->
 <joint name="caster_wheel_joint" type="fixed">
@@ -107,3 +116,8 @@
     </xacro:inertial_sphere>
 </link>
+<gazebo reference="caster_wheel">
+    <material>Gazebo/Black</material>
+    <mu1 value="0.001"/>
+    <mu2 value="0.001"/>
+</gazebo>
 </robot>

Commit message: red color lidar added

File: description/robot.urdf.xacro (robot description, xacro)
@@ -3,3 +3,4 @@
     <xacro:include filename = "robot_core.xacro"/>
     <xacro:include filename = "gazebo_control.xacro"/>
+    <xacro:include filename = "lidar.xacro"/>
 </robot>

File: description/robot_core.xacro (robot description, xacro)
@@ -13,4 +13,7 @@
     <material name="black">
         <color rgba="0 0 0 1"/>
+    </material>
+    <material name="red">
+        <color rgba="1 0 0 1"/>
     </material>
     <link name="base_link">

Commit message: updated and gazebo fixes

File: description/robot.urdf.xacro (robot description, xacro)
@@ -2,5 +2,6 @@
 <robot xmlns:xacro="http://www.ros.org/wiki/xacro"  name="robot">
     <xacro:include filename = "robot_core.xacro"/>
-    <xacro:include filename = "gazebo_control.xacro"/>
+    <xacro:include filename = "ros2_control.xacro"/>
+    <!-- <xacro:include filename = "gazebo_control.xacro"/>  -->
     <xacro:include filename = "lidar.xacro"/>
 </robot>

File: description/robot_core.xacro (robot description, xacro)
@@ -61,5 +61,5 @@
     <collision>
         <geometry>
-            <cylinder length="0.04" radius="0.05" />
+            <sphere radius="0.05" />
         </geometry>
     </collision>
@@ -87,5 +87,5 @@
     <collision>
         <geometry>
-            <cylinder length="0.04" radius="0.05" />
+            <sphere radius="0.05" />
         </geometry>
     </collision>

Commit message: nav2 humble

File: description/robot.urdf.xacro (robot description, xacro)
@@ -1,7 +1,12 @@
 <?xml version="1.0"?>
 <robot xmlns:xacro="http://www.ros.org/wiki/xacro"  name="robot">
+    <xacro:arg name="use_ros2_control" default="true"/>
     <xacro:include filename = "robot_core.xacro"/>
-    <xacro:include filename = "ros2_control.xacro"/>
-    <!-- <xacro:include filename = "gazebo_control.xacro"/>  -->
+    <xacro:if value="$(arg use_ros2_control)">
+        <xacro:include filename = "ros2_control.xacro"/>
+    </xacro:if>
+    <xacro:unless value="$(arg use_ros2_control)">
+        <xacro:include filename = "gazebo_control.xacro"/>
+    </xacro:unless>
     <xacro:include filename = "lidar.xacro"/>
 </robot>

File: description/robot_core.xacro (robot description, xacro)
@@ -18,4 +18,11 @@
     </material>
     <link name="base_link">
+    </link>
+    <joint name ="base_footprint_link" type="fixed">
+        <parent link="base_link"/>
+        <child link="base_footprint"/>
+        <origin xyz ="0 0 0" rpy ="0 0 0"/>
+    </joint>
+    <link name="base_footprint">
     </link>
     <joint name="chassis_joint" type="fixed">
